File: spectrometerbreakout.kicad_sch (KiCad schematic)
At the start: 0 parts

Commit message: changed naming conventions
Parts:
- added C1, C2: 10uF, symbol Device:C
- added C10, C12: C, symbol Device:C
- added C11: 1nF, symbol Device:C
- added C3: 1uF, symbol Device:C
- added C4: 100nF, symbol Device:C
- added C5: 1kuF, symbol Device:C
- added C6: 39nF, symbol Device:C
- added C7: 0.47uF, symbol Device:C
- added C8: 2.2uF, symbol Device:C
- added C9: 47uF, symbol Device:C
- added R1, R4: 1k, symbol Device:R
- added R2, R3, R8: 10k, symbol Device:R
- added R5: 500, symbol Device:R
- added R6: 10, symbol Device:R
- added R7: R, symbol Device:R
- added U1: C12880MA, OptoDevice:Hamamatsu_C12880, symbol Sensor_Optical:C12880MA
- added U2, U5, U7: OPA365xxD, Package_SO:SOIC-8_3.9x4.9mm_P1.27mm, symbol Amplifier_Operational:OPA365xxD
- added U3: ADS8326, symbol ADSxxxx:ADS8326
- added U4: RP2350B, Package_DFN_QFN:QFN-80-1EP_10x10mm_P0.4mm_EP3.4x3.4mm, symbol MCU_RaspberryPi:RP2350B
- added U6: REF3225AMDBVREP, Package_TO_SOT_SMD:SOT-23-6, symbol Reference_Voltage:REF3225AMDBVREP
Connections:
- new net: C12.1, U7.7 (V+)
- new net: C1.1, C2.1, U1.1 (VCC), U1.3 (VCC)
- new net: C8.2, C9.2, R6.2, U3.1 (REF), U5.3 (+), U5.6
- new net: C3.2, U3.8 (VDD)
- new net: R3.2, R5.2, U2.3 (+)
- new net: R3.1, R4.2, U2.6
- new net: C4.1, U2.7 (V+)
- new net: C7.1, U6.3 (ENABLE)
- new net: R7.2, R8.2, U7.6
- new net: C6.1, R2.2, R5.1
- new net: R6.1, U6.5 (OUT_S), U6.6 (OUT_F)
- new net: C11.2, C5.1, R4.1, U3.2 (+IN)
- new net: C10.1, C11.1, R7.1, U3.3 (-IN)
- new net: U4.10 (DVDD), U4.32 (DVDD), U4.51 (DVDD)
- new net: U4.15 (IOVDD), U4.24 (IOVDD), U4.29 (IOVDD), U4.41 (IOVDD), U4.5 (IOVDD), U4.50 (IOVDD), U4.60 (IOVDD), U4.76 (IOVDD)
- new net: R2.1, U1.10 (VIDEO)
- new net: R1.2, U1.4 (CLK)
- new net GND: C1.2, C10.2, C12.2, C2.2, C4.2, C5.2, C6.2, C7.2, C8.1, C9.1, U1.2 (GND), U1.5 (CASE), U2.2 (-), U2.4 (V-), U3.4 (GND), U3.5 (CS/SHDN), U5.2 (-), U5.4 (V-), U6.1 (GNDF), U6.2 (GNDS), U6.4 (VIN), U7.2 (-), U7.4 (V-)
- new net GPIO0: R1.1
- new net GPIO1: U1.7 (TRG)
- new net GPIO2: U1.9 (EOS)
- new net GPIO3: U3.6 (D_OUT)
- new net QSPI_SCLK: U3.7 (DCLOCK)
- new net VCM?: R8.1, U7.3 (+)
Other:
- company: (none) -> BoilerRobotics/Lunabotics
- title: (none) -> Spectrometer Breakout Board
